Commit message: add Isaac Lab sim, fix URDF mesh paths, track meshes in repo

File: assets/iRonCub/robots/iRonCub-Mk1_1/model.urdf (robot description, URDF)
Before this commit: robot iCub, 97 links, 96 joints
Links:
- link chest: geometry collision mesh filename=../../meshes/obj/sim_sea_2-5_chest_bb_prt.obj scale=0.001 0.001 0.001; visual mesh filename=../../meshes/obj/sim_sea_2-5_chest_bb_prt.obj scale=0.001 0.001 0.001
- link chest_aruco_origin: geometry collision mesh filename=../../meshes/obj/sim_sea_2-5_chest_aruco_prt.obj scale=0.001 0.001 0.001; visual mesh filename=../../meshes/obj/sim_sea_2-5_chest_aruco_prt.obj scale=0.001 0.001 0.001
- link chest_l_jet_turbine: geometry collision mesh filename=../../meshes/obj/sim_sea_2-5_l_p220_prt.obj scale=0.001 0.001 0.001; visual mesh filename=../../meshes/obj/sim_sea_2-5_l_p220_prt.obj scale=0.001 0.001 0.001
- link chest_r_jet_turbine: geometry collision mesh filename=../../meshes/obj/sim_sea_2-5_r_p220_prt.obj scale=0.001 0.001 0.001; visual mesh filename=../../meshes/obj/sim_sea_2-5_r_p220_prt.obj scale=0.001 0.001 0.001
- link head: geometry collision mesh filename=../../meshes/obj/sim_sea_2-5_head_prt.obj scale=0.001 0.001 0.001; visual mesh filename=../../meshes/obj/sim_sea_2-5_head_prt.obj scale=0.001 0.001 0.001
- link l_ankle_1: geometry collision mesh filename=../../meshes/obj/sim_sea_2-5_l_ankle_prt.obj scale=0.001 0.001 0.001; visual mesh filename=../../meshes/obj/sim_sea_2-5_l_ankle_prt.obj scale=0.001 0.001 0.001
- link l_ankle_2: geometry collision mesh filename=../../meshes/obj/sim_sea_2-5_l_foot_prt.obj scale=0.001 0.001 0.001; visual mesh filename=../../meshes/obj/sim_sea_2-5_l_foot_prt.obj scale=0.001 0.001 0.001
- link l_arm_jet_turbine: geometry collision mesh filename=../../meshes/obj/sim_sea_2-5_l_elbow_p160_prt.obj scale=0.001 0.001 0.001; visual mesh filename=../../meshes/obj/sim_sea_2-5_l_elbow_p160_prt.obj scale=0.001 0.001 0.001
- link l_elbow_1: geometry collision mesh filename=../../meshes/obj/sim_sea_2-5_l_elbow_prosup_prt.obj scale=0.001 0.001 0.001; visual mesh filename=../../meshes/obj/sim_sea_2-5_l_elbow_prosup_prt.obj scale=0.001 0.001 0.001
- link l_foot: geometry collision mesh filename=../../meshes/obj/sim_sea_2-5_l_sole_prt.obj scale=0.001 0.001 0.001; visual mesh filename=../../meshes/obj/sim_sea_2-5_l_sole_prt.obj scale=0.001 0.001 0.001
- link l_hip_1: geometry collision mesh filename=../../meshes/obj/sim_sea_2-5_l_hip_1_prt.obj scale=0.001 0.001 0.001; visual mesh filename=../../meshes/obj/sim_sea_2-5_l_hip_1_prt.obj scale=0.001 0.001 0.001
- link l_hip_2: geometry collision mesh filename=../../meshes/obj/sim_sea_2-5_l_hip_2_prt.obj scale=0.001 0.001 0.001; visual mesh filename=../../meshes/obj/sim_sea_2-5_l_hip_2_prt.obj scale=0.001 0.001 0.001
- link l_hip_3: geometry collision mesh filename=../../meshes/obj/sim_sea_2-5_l_upper_thigh_prt.obj scale=0.001 0.001 0.001; visual mesh filename=../../meshes/obj/sim_sea_2-5_l_upper_thigh_prt.obj scale=0.001 0.001 0.001
- link l_lower_leg: geometry collision mesh filename=../../meshes/obj/sim_sea_2-5_l_shank_prt.obj scale=0.001 0.001 0.001; visual mesh filename=../../meshes/obj/sim_sea_2-5_l_shank_prt.obj scale=0.001 0.001 0.001
- link l_shoulder_1: geometry collision mesh filename=../../meshes/obj/sim_sea_2-5_l_shoulder_1_prt.obj scale=0.001 0.001 0.001; visual mesh filename=../../meshes/obj/sim_sea_2-5_l_shoulder_1_prt.obj scale=0.001 0.001 0.001
- link l_shoulder_2: geometry collision mesh filename=../../meshes/obj/sim_sea_2-5_l_shoulder_2_prt.obj scale=0.001 0.001 0.001; visual mesh filename=../../meshes/obj/sim_sea_2-5_l_shoulder_2_prt.obj scale=0.001 0.001 0.001
- link l_shoulder_3: geometry collision mesh filename=../../meshes/obj/sim_sea_2-5_l_upper_arm_prt.obj scale=0.001 0.001 0.001; visual mesh filename=../../meshes/obj/sim_sea_2-5_l_upper_arm_prt.obj scale=0.001 0.001 0.001
- link l_upper_arm: geometry collision mesh filename=../../meshes/obj/sim_sea_2-5_l_elbow_prt.obj scale=0.001 0.001 0.001; visual mesh filename=../../meshes/obj/sim_sea_2-5_l_elbow_prt.obj scale=0.001 0.001 0.001
- link l_upper_leg: geometry collision mesh filename=../../meshes/obj/sim_sea_2-5_l_thigh_prt.obj scale=0.001 0.001 0.001; visual mesh filename=../../meshes/obj/sim_sea_2-5_l_thigh_prt.obj scale=0.001 0.001 0.001
- link neck_1: geometry collision mesh filename=../../meshes/obj/sim_sea_2-5_neck_1_prt.obj scale=0.001 0.001 0.001; visual mesh filename=../../meshes/obj/sim_sea_2-5_neck_1_prt.obj scale=0.001 0.001 0.001
- link neck_2: geometry collision mesh filename=../../meshes/obj/sim_sea_2-5_neck_2_prt.obj scale=0.001 0.001 0.001; visual mesh filename=../../meshes/obj/sim_sea_2-5_neck_2_prt.obj scale=0.001 0.001 0.001
- link r_ankle_1: geometry collision mesh filename=../../meshes/obj/sim_sea_2-5_r_ankle_prt.obj scale=0.001 0.001 0.001; visual mesh filename=../../meshes/obj/sim_sea_2-5_r_ankle_prt.obj scale=0.001 0.001 0.001
- link r_ankle_2: geometry collision mesh filename=../../meshes/obj/sim_sea_2-5_r_foot_prt.obj scale=0.001 0.001 0.001; visual mesh filename=../../meshes/obj/sim_sea_2-5_r_foot_prt.obj scale=0.001 0.001 0.001
- link r_arm_jet_turbine: geometry collision mesh filename=../../meshes/obj/sim_sea_2-5_r_elbow_p160_prt.obj scale=0.001 0.001 0.001; visual mesh filename=../../meshes/obj/sim_sea_2-5_r_elbow_p160_prt.obj scale=0.001 0.001 0.001
- link r_elbow_1: geometry collision mesh filename=../../meshes/obj/sim_sea_2-5_r_elbow_prosup_prt.obj scale=0.001 0.001 0.001; visual mesh filename=../../meshes/obj/sim_sea_2-5_r_elbow_prosup_prt.obj scale=0.001 0.001 0.001
- link r_foot: geometry collision mesh filename=../../meshes/obj/sim_sea_2-5_r_sole_prt.obj scale=0.001 0.001 0.001; visual mesh filename=../../meshes/obj/sim_sea_2-5_r_sole_prt.obj scale=0.001 0.001 0.001
- link r_hip_1: geometry collision mesh filename=../../meshes/obj/sim_sea_2-5_r_hip_1_prt.obj scale=0.001 0.001 0.001; visual mesh filename=../../meshes/obj/sim_sea_2-5_r_hip_1_prt.obj scale=0.001 0.001 0.001
- link r_hip_2: geometry collision mesh filename=../../meshes/obj/sim_sea_2-5_r_hip_2_prt.obj scale=0.001 0.001 0.001; visual mesh filename=../../meshes/obj/sim_sea_2-5_r_hip_2_prt.obj scale=0.001 0.001 0.001
- link r_hip_3: geometry collision mesh filename=../../meshes/obj/sim_sea_2-5_r_upper_thigh_prt.obj scale=0.001 0.001 0.001; visual mesh filename=../../meshes/obj/sim_sea_2-5_r_upper_thigh_prt.obj scale=0.001 0.001 0.001
- link r_lower_leg: geometry collision mesh filename=../../meshes/obj/sim_sea_2-5_r_shank_prt.obj scale=0.001 0.001 0.001; visual mesh filename=../../meshes/obj/sim_sea_2-5_r_shank_prt.obj scale=0.001 0.001 0.001
- link r_shoulder_1: geometry collision mesh filename=../../meshes/obj/sim_sea_2-5_r_shoulder_1_prt.obj scale=0.001 0.001 0.001; visual mesh filename=../../meshes/obj/sim_sea_2-5_r_shoulder_1_prt.obj scale=0.001 0.001 0.001
- link r_shoulder_2: geometry collision mesh filename=../../meshes/obj/sim_sea_2-5_r_shoulder_2_prt.obj scale=0.001 0.001 0.001; visual mesh filename=../../meshes/obj/sim_sea_2-5_r_shoulder_2_prt.obj scale=0.001 0.001 0.001
- link r_shoulder_3: geometry collision mesh filename=../../meshes/obj/sim_sea_2-5_r_upper_arm_prt.obj scale=0.001 0.001 0.001; visual mesh filename=../../meshes/obj/sim_sea_2-5_r_upper_arm_prt.obj scale=0.001 0.001 0.001
- link r_upper_arm: geometry collision mesh filename=../../meshes/obj/sim_sea_2-5_r_elbow_prt.obj scale=0.001 0.001 0.001; visual mesh filename=../../meshes/obj/sim_sea_2-5_r_elbow_prt.obj scale=0.001 0.001 0.001
- link r_upper_leg: geometry collision mesh filename=../../meshes/obj/sim_sea_2-5_r_thigh_prt.obj scale=0.001 0.001 0.001; visual mesh filename=../../meshes/obj/sim_sea_2-5_r_thigh_prt.obj scale=0.001 0.001 0.001
- link root_link: geometry collision mesh filename=../../meshes/obj/sim_sea_2-5_root_link_prt.obj scale=0.001 0.001 0.001; visual mesh filename=../../meshes/obj/sim_sea_2-5_root_link_prt.obj scale=0.001 0.001 0.001
- link torso_1: geometry collision mesh filename=../../meshes/obj/sim_sea_2-5_lap_belt_1_prt.obj scale=0.001 0.001 0.001; visual mesh filename=../../meshes/obj/sim_sea_2-5_lap_belt_1_prt.obj scale=0.001 0.001 0.001
- link torso_2: geometry collision mesh filename=../../meshes/obj/sim_sea_2-5_lap_belt_2_prt.obj scale=0.001 0.001 0.001; visual mesh filename=../../meshes/obj/sim_sea_2-5_lap_belt_2_prt.obj scale=0.001 0.001 0.001

File: assets/iRonCub/robots/iRonCub-Mk1_1/model_stl.urdf (robot description, URDF)
Before this commit: robot iCub, 97 links, 96 joints
Links:
- link chest: geometry collision mesh filename=../../meshes/stl/sim_sea_2-5_chest_bb_prt.stl scale=0.001 0.001 0.001; visual mesh filename=../../meshes/stl/sim_sea_2-5_chest_bb_prt.stl scale=0.001 0.001 0.001
- link chest_aruco_origin: geometry collision mesh filename=../../meshes/stl/sim_sea_2-5_chest_aruco_prt.stl scale=0.001 0.001 0.001; visual mesh filename=../../meshes/stl/sim_sea_2-5_chest_aruco_prt.stl scale=0.001 0.001 0.001
- link chest_l_jet_turbine: geometry collision mesh filename=../../meshes/stl/sim_sea_2-5_l_p220_prt.stl scale=0.001 0.001 0.001; visual mesh filename=../../meshes/stl/sim_sea_2-5_l_p220_prt.stl scale=0.001 0.001 0.001
- link chest_r_jet_turbine: geometry collision mesh filename=../../meshes/stl/sim_sea_2-5_r_p220_prt.stl scale=0.001 0.001 0.001; visual mesh filename=../../meshes/stl/sim_sea_2-5_r_p220_prt.stl scale=0.001 0.001 0.001
- link head: geometry collision mesh filename=../../meshes/stl/sim_sea_2-5_head_prt.stl scale=0.001 0.001 0.001; visual mesh filename=../../meshes/stl/sim_sea_2-5_head_prt.stl scale=0.001 0.001 0.001
- link l_ankle_1: geometry collision mesh filename=../../meshes/stl/sim_sea_2-5_l_ankle_prt.stl scale=0.001 0.001 0.001; visual mesh filename=../../meshes/stl/sim_sea_2-5_l_ankle_prt.stl scale=0.001 0.001 0.001
- link l_ankle_2: geometry collision mesh filename=../../meshes/stl/sim_sea_2-5_l_foot_prt.stl scale=0.001 0.001 0.001; visual mesh filename=../../meshes/stl/sim_sea_2-5_l_foot_prt.stl scale=0.001 0.001 0.001
- link l_arm_jet_turbine: geometry collision mesh filename=../../meshes/stl/sim_sea_2-5_l_elbow_p160_prt.stl scale=0.001 0.001 0.001; visual mesh filename=../../meshes/stl/sim_sea_2-5_l_elbow_p160_prt.stl scale=0.001 0.001 0.001
- link l_elbow_1: geometry collision mesh filename=../../meshes/stl/sim_sea_2-5_l_elbow_prosup_prt.stl scale=0.001 0.001 0.001; visual mesh filename=../../meshes/stl/sim_sea_2-5_l_elbow_prosup_prt.stl scale=0.001 0.001 0.001
- link l_foot: geometry collision mesh filename=../../meshes/stl/sim_sea_2-5_l_sole_prt.stl scale=0.001 0.001 0.001; visual mesh filename=../../meshes/stl/sim_sea_2-5_l_sole_prt.stl scale=0.001 0.001 0.001
- link l_hip_1: geometry collision mesh filename=../../meshes/stl/sim_sea_2-5_l_hip_1_prt.stl scale=0.001 0.001 0.001; visual mesh filename=../../meshes/stl/sim_sea_2-5_l_hip_1_prt.stl scale=0.001 0.001 0.001
- link l_hip_2: geometry collision mesh filename=../../meshes/stl/sim_sea_2-5_l_hip_2_prt.stl scale=0.001 0.001 0.001; visual mesh filename=../../meshes/stl/sim_sea_2-5_l_hip_2_prt.stl scale=0.001 0.001 0.001
- link l_hip_3: geometry collision mesh filename=../../meshes/stl/sim_sea_2-5_l_upper_thigh_prt.stl scale=0.001 0.001 0.001; visual mesh filename=../../meshes/stl/sim_sea_2-5_l_upper_thigh_prt.stl scale=0.001 0.001 0.001
- link l_lower_leg: geometry collision mesh filename=../../meshes/stl/sim_sea_2-5_l_shank_prt.stl scale=0.001 0.001 0.001; visual mesh filename=../../meshes/stl/sim_sea_2-5_l_shank_prt.stl scale=0.001 0.001 0.001
- link l_shoulder_1: geometry collision mesh filename=../../meshes/stl/sim_sea_2-5_l_shoulder_1_prt.stl scale=0.001 0.001 0.001; visual mesh filename=../../meshes/stl/sim_sea_2-5_l_shoulder_1_prt.stl scale=0.001 0.001 0.001
- link l_shoulder_2: geometry collision mesh filename=../../meshes/stl/sim_sea_2-5_l_shoulder_2_prt.stl scale=0.001 0.001 0.001; visual mesh filename=../../meshes/stl/sim_sea_2-5_l_shoulder_2_prt.stl scale=0.001 0.001 0.001
- link l_shoulder_3: geometry collision mesh filename=../../meshes/stl/sim_sea_2-5_l_upper_arm_prt.stl scale=0.001 0.001 0.001; visual mesh filename=../../meshes/stl/sim_sea_2-5_l_upper_arm_prt.stl scale=0.001 0.001 0.001
- link l_upper_arm: geometry collision mesh filename=../../meshes/stl/sim_sea_2-5_l_elbow_prt.stl scale=0.001 0.001 0.001; visual mesh filename=../../meshes/stl/sim_sea_2-5_l_elbow_prt.stl scale=0.001 0.001 0.001
- link l_upper_leg: geometry collision mesh filename=../../meshes/stl/sim_sea_2-5_l_thigh_prt.stl scale=0.001 0.001 0.001; visual mesh filename=../../meshes/stl/sim_sea_2-5_l_thigh_prt.stl scale=0.001 0.001 0.001
- link neck_1: geometry collision mesh filename=../../meshes/stl/sim_sea_2-5_neck_1_prt.stl scale=0.001 0.001 0.001; visual mesh filename=../../meshes/stl/sim_sea_2-5_neck_1_prt.stl scale=0.001 0.001 0.001
- link neck_2: geometry collision mesh filename=../../meshes/stl/sim_sea_2-5_neck_2_prt.stl scale=0.001 0.001 0.001; visual mesh filename=../../meshes/stl/sim_sea_2-5_neck_2_prt.stl scale=0.001 0.001 0.001
- link r_ankle_1: geometry collision mesh filename=../../meshes/stl/sim_sea_2-5_r_ankle_prt.stl scale=0.001 0.001 0.001; visual mesh filename=../../meshes/stl/sim_sea_2-5_r_ankle_prt.stl scale=0.001 0.001 0.001
- link r_ankle_2: geometry collision mesh filename=../../meshes/stl/sim_sea_2-5_r_foot_prt.stl scale=0.001 0.001 0.001; visual mesh filename=../../meshes/stl/sim_sea_2-5_r_foot_prt.stl scale=0.001 0.001 0.001
- link r_arm_jet_turbine: geometry collision mesh filename=../../meshes/stl/sim_sea_2-5_r_elbow_p160_prt.stl scale=0.001 0.001 0.001; visual mesh filename=../../meshes/stl/sim_sea_2-5_r_elbow_p160_prt.stl scale=0.001 0.001 0.001
- link r_elbow_1: geometry collision mesh filename=../../meshes/stl/sim_sea_2-5_r_elbow_prosup_prt.stl scale=0.001 0.001 0.001; visual mesh filename=../../meshes/stl/sim_sea_2-5_r_elbow_prosup_prt.stl scale=0.001 0.001 0.001
- link r_foot: geometry collision mesh filename=../../meshes/stl/sim_sea_2-5_r_sole_prt.stl scale=0.001 0.001 0.001; visual mesh filename=../../meshes/stl/sim_sea_2-5_r_sole_prt.stl scale=0.001 0.001 0.001
- link r_hip_1: geometry collision mesh filename=../../meshes/stl/sim_sea_2-5_r_hip_1_prt.stl scale=0.001 0.001 0.001; visual mesh filename=../../meshes/stl/sim_sea_2-5_r_hip_1_prt.stl scale=0.001 0.001 0.001
- link r_hip_2: geometry collision mesh filename=../../meshes/stl/sim_sea_2-5_r_hip_2_prt.stl scale=0.001 0.001 0.001; visual mesh filename=../../meshes/stl/sim_sea_2-5_r_hip_2_prt.stl scale=0.001 0.001 0.001
- link r_hip_3: geometry collision mesh filename=../../meshes/stl/sim_sea_2-5_r_upper_thigh_prt.stl scale=0.001 0.001 0.001; visual mesh filename=../../meshes/stl/sim_sea_2-5_r_upper_thigh_prt.stl scale=0.001 0.001 0.001
- link r_lower_leg: geometry collision mesh filename=../../meshes/stl/sim_sea_2-5_r_shank_prt.stl scale=0.001 0.001 0.001; visual mesh filename=../../meshes/stl/sim_sea_2-5_r_shank_prt.stl scale=0.001 0.001 0.001
- link r_shoulder_1: geometry collision mesh filename=../../meshes/stl/sim_sea_2-5_r_shoulder_1_prt.stl scale=0.001 0.001 0.001; visual mesh filename=../../meshes/stl/sim_sea_2-5_r_shoulder_1_prt.stl scale=0.001 0.001 0.001
- link r_shoulder_2: geometry collision mesh filename=../../meshes/stl/sim_sea_2-5_r_shoulder_2_prt.stl scale=0.001 0.001 0.001; visual mesh filename=../../meshes/stl/sim_sea_2-5_r_shoulder_2_prt.stl scale=0.001 0.001 0.001
- link r_shoulder_3: geometry collision mesh filename=../../meshes/stl/sim_sea_2-5_r_upper_arm_prt.stl scale=0.001 0.001 0.001; visual mesh filename=../../meshes/stl/sim_sea_2-5_r_upper_arm_prt.stl scale=0.001 0.001 0.001
- link r_upper_arm: geometry collision mesh filename=../../meshes/stl/sim_sea_2-5_r_elbow_prt.stl scale=0.001 0.001 0.001; visual mesh filename=../../meshes/stl/sim_sea_2-5_r_elbow_prt.stl scale=0.001 0.001 0.001
- link r_upper_leg: geometry collision mesh filename=../../meshes/stl/sim_sea_2-5_r_thigh_prt.stl scale=0.001 0.001 0.001; visual mesh filename=../../meshes/stl/sim_sea_2-5_r_thigh_prt.stl scale=0.001 0.001 0.001
- link root_link: geometry collision mesh filename=../../meshes/stl/sim_sea_2-5_root_link_prt.stl scale=0.001 0.001 0.001; visual mesh filename=../../meshes/stl/sim_sea_2-5_root_link_prt.stl scale=0.001 0.001 0.001
- link torso_1: geometry collision mesh filename=../../meshes/stl/sim_sea_2-5_lap_belt_1_prt.stl scale=0.001 0.001 0.001; visual mesh filename=../../meshes/stl/sim_sea_2-5_lap_belt_1_prt.stl scale=0.001 0.001 0.001
- link torso_2: geometry collision mesh filename=../../meshes/stl/sim_sea_2-5_lap_belt_2_prt.stl scale=0.001 0.001 0.001; visual mesh filename=../../meshes/stl/sim_sea_2-5_lap_belt_2_prt.stl scale=0.001 0.001 0.001
